File: cpu.kicad_sch (KiCad schematic)
At the start: 0 parts

Commit message: updates
Parts:
- added R10, R11, R12, R13, R14, R21, R22, R23, R24, R25, R26, R9: 4.7k, Resistor_SMD:R_0201_0603Metric, symbol Device:R
- added U6: 68000D, Package_DIP:DIP-64_W25.4mm_Socket, symbol CPU_NXP_68000:68000D
Connections:
- new net +5V: R10.2, R11.2, R12.2, R13.2, R14.2, R21.2, R22.2, R23.2, R24.2, R25.2, R26.2, R9.2
- new net A1: U6.29 (A1)
- new net A10: U6.38 (A10)
- new net A11: U6.39 (A11)
- new net A12: U6.40 (A12)
- new net A13: U6.41 (A13)
- new net A14: U6.42 (A14)
- new net A15: U6.43 (A15)
- new net A16: U6.44 (A16)
- new net A17: U6.45 (A17)
- new net A18: U6.46 (A18)
- new net A19: U6.47 (A19)
- new net A2: U6.30 (A2)
- new net A20: U6.48 (A20)
- new net A21: U6.50 (A21)
- new net A22: U6.51 (A22)
- new net A23: U6.52 (A23)
- new net A3: U6.31 (A3)
- new net A4: U6.32 (A4)
- new net A5: U6.33 (A5)
- new net A6: U6.34 (A6)
- new net A7: U6.35 (A7)
- new net A8: U6.36 (A8)
- new net A9: U6.37 (A9)
- new net AS: U6.6 (AS)
- new net BG: R13.1, U6.11 (BG)
- new net BGACK: R12.1, U6.12 (BGACK)
- new net BR: R14.1, U6.13 (BR)
- new net CLOCK: U6.15 (CLK)
- new net D0: U6.5 (D0)
- new net D1: U6.4 (D1)
- new net D10: U6.59 (D10)
- new net D11: U6.58 (D11)
- new net D12: U6.57 (D12)
- new net D13: U6.56 (D13)
- new net D14: U6.55 (D14)
- new net D15: U6.54 (D15)
- new net D2: U6.3 (D2)
- new net D3: U6.2 (D3)
- new net D4: U6.1 (D4)
- new net D5: U6.64 (D5)
- new net D6: U6.63 (D6)
- new net D7: U6.62 (D7)
- new net D8: U6.61 (D8)
- new net D9: U6.60 (D9)
- new net E: R25.1, U6.20 (E)
- new net FC0: R21.1, U6.28 (FC0)
- new net FC1: R22.1, U6.27 (FC1)
- new net FC2: R23.1, U6.26 (FC2)
- new net IPL0: R9.1, U6.25 (IPL0)
- new net IPL1: R10.1, U6.24 (IPL1)
- new net IPL2: R11.1, U6.23 (IPL2)
- new net LDS: U6.8 (LDS)
- new net RW: U6.9 (R/W)
- new net UDS: U6.7 (UDS)
- new net VMA: R24.1, U6.19 (VMA)
- new net VPA: R26.1, U6.21 (VPA)
- new net ~{BERR}: U6.22 (BERR)
- new net ~{DTACK}: U6.10 (DTACK)
- new net ~{HALT}: U6.17 (HALT)
- new net ~{RESET}: U6.18 (RESET)
Other:
- note added: "A20 is RAM CE A21 is Pseudo ROM A22 is Pseudo IO"

Commit message: updates
Changed lines of the file:
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@@
     (stroke (width 0) (type default))
   )
-  (text "A20 is RAM CE\nA21 is Pseudo ROM\nA22 is Pseudo IO" (at 209.55 82.55 0)
+  (text "A20 is RAM CE\nA21 is Pseudo ROM\nA22 is Pseudo IO" (at 212.09 82.55 0)
     (effects (font (size 1.27 1.27)) (justify left bottom))
   )
