File: power.kicad_sch (KiCad schematic)
At the start: 20 parts, among them J1 USB_B_Micro_Console, J4 USB_B_Micro_Power, U1 SRV05-4

Commit message: updates
Parts:
- removed TP2, TP5: TestPoint, TestPoint:TestPoint_Pad_D1.5mm, symbol Connector:TestPoint
- added TP6: TestPoint, TestPoint:TestPoint_Pad_D1.5mm, symbol Connector:TestPoint
- added TP7: TestPoint, TestPoint:TestPoint_Pad_1.5x1.5mm, symbol Connector:TestPoint
Connections:
- net +5V is gone; now on net VCC: C7.1, C8.1, FB2.1, R2.1
- net GND: now also TP7.1
- net USB_VBUS: no longer TP4.1
- net VCC: now also TP4.1, TP6.1
Other:
- moved on the sheet: C1, C2, C3, D1, FB1, J1, J4, R1, TP1, TP4

Commit message: updates
Parts:
- removed TP3: TestPoint, TestPoint:TestPoint_Pad_D1.5mm, symbol Connector:TestPoint
Changed lines of the file:
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@@
-    )
-  )
-  (global_label "USB_VBUS" (shape input) (at 46.99 167.64 180) (fields_autoplaced)
-    (effects (font (size 1.27 1.27)) (justify right))
-    (property "Intersheetrefs" "${INTERSHEET_REFS}" (at 34.3286 167.64 0)
-      (effects (font (size 1.27 1.27)) (justify right) hide)
     )
   )
@@
     )
   )
-  (global_label "USB_POWER" (shape input) (at 46.99 176.53 180) (fields_autoplaced)
-    (effects (font (size 1.27 1.27)) (justify right))
-    (property "Intersheetrefs" "${INTERSHEET_REFS}" (at 32.7563 176.53 0)
-      (effects (font (size 1.27 1.27)) (justify right) hide)
-    )
-  )
   (global_label "USB_VBUS" (shape output) (at 147.32 29.21 180) (fields_autoplaced)
     (effects (font (size 1.27 1.27)) (justify right))
@@
     )
   )
+  (symbol (lib_id "power:PWR_FLAG") (at 223.52 134.62 270) (unit 1)
+    (in_bom yes) (on_board yes) (dnp no) (fields_autoplaced)
+    (property "Reference" "#FLG04" (at 225.425 134.62 0)
+      (effects (font (size 1.27 1.27)) hide)
+    )
+    (property "Value" "PWR_FLAG" (at 227.33 134.62 90)
+      (effects (font (size 1.27 1.27)) (justify left))
+    )
+    (property "Footprint" "" (at 223.52 134.62 0)
+      (effects (font (size 1.27 1.27)) hide)
+    )
+    (property "Datasheet" "~" (at 223.52 134.62 0)
+      (effects (font (size 1.27 1.27)) hide)
+    )
+    (pin "1")
+    (instances
+      (project "leo68k"
+        (path "/33088729-b62e-4c27-bd07-0e3dd7f7f61e/3f60a7ce-0238-4481-8009-2dff3c5599e1"
+          (reference "#FLG04") (unit 1)
+        )
+      )
+    )
+  )
+  (symbol (lib_id "power:PWR_FLAG") (at 223.52 109.22 270) (unit 1)
+    (in_bom yes) (on_board yes) (dnp no) (fields_autoplaced)
+    (property "Reference" "#FLG03" (at 225.425 109.22 0)
+      (effects (font (size 1.27 1.27)) hide)
+    )
+    (property "Value" "PWR_FLAG" (at 227.33 109.22 90)
+      (effects (font (size 1.27 1.27)) (justify left))
+    )
+    (property "Footprint" "" (at 223.52 109.22 0)
+      (effects (font (size 1.27 1.27)) hide)
+    )
+    (property "Datasheet" "~" (at 223.52 109.22 0)
+      (effects (font (size 1.27 1.27)) hide)
+    )
+    (pin "1")
+    (instances
+      (project "leo68k"
+        (path "/33088729-b62e-4c27-bd07-0e3dd7f7f61e/3f60a7ce-0238-4481-8009-2dff3c5599e1"
+          (reference "#FLG03") (unit 1)
+        )
+      )
+    )
+  )
   (symbol (lib_id "power:GND") (at 223.52 59.69 0) (unit 1)
     (in_bom yes) (on_board yes) (dnp no) (fields_autoplaced)
@@
     )
   )
-  (symbol (lib_id "Connector:TestPoint") (at 46.99 176.53 0) (unit 1)
-    (in_bom yes) (on_board yes) (dnp no)
-    (property "Reference" "TP3" (at 49.53 171.958 0)
-      (effects (font (size 1.27 1.27)) (justify left))
-    )
-    (property "Value" "TestPoint" (at 49.53 174.498 0)
-      (effects (font (size 1.27 1.27)) (justify left))
-    )
-    (property "Footprint" "TestPoint:TestPoint_Pad_D1.5mm" (at 52.07 176.53 0)
-      (effects (font (size 1.27 1.27)) hide)
-    )
-    (property "Datasheet" "~" (at 52.07 176.53 0)
-      (effects (font (size 1.27 1.27)) hide)
-    )
-    (property "JLPCB Part" "" (at 46.99 176.53 0)
-      (effects (font (size 1.27 1.27)) hide)
-    )
-    (pin "1")
-    (instances
-      (project "leo68k"
-        (path "/33088729-b62e-4c27-bd07-0e3dd7f7f61e/3f60a7ce-0238-4481-8009-2dff3c5599e1"
-          (reference "TP3") (unit 1)
+  (symbol (lib_id "power:PWR_FLAG") (at 223.52 29.21 270) (unit 1)
+    (in_bom yes) (on_board yes) (dnp no) (fields_autoplaced)
+    (property "Reference" "#FLG01" (at 225.425 29.21 0)
+      (effects (font (size 1.27 1.27)) hide)
+    )
+    (property "Value" "PWR_FLAG" (at 227.33 29.21 90)
+      (effects (font (size 1.27 1.27)) (justify left))
+    )
+    (property "Footprint" "" (at 223.52 29.21 0)
+      (effects (font (size 1.27 1.27)) hide)
+    )
+    (property "Datasheet" "~" (at 223.52 29.21 0)
+      (effects (font (size 1.27 1.27)) hide)
+    )
+    (pin "1")
+    (instances
+      (project "leo68k"
+        (path "/33088729-b62e-4c27-bd07-0e3dd7f7f61e/3f60a7ce-0238-4481-8009-2dff3c5599e1"
+          (reference "#FLG01") (unit 1)
         )
       )
@@
         )
       )
+    )
+  )
+  (symbol (lib_id "power:PWR_FLAG") (at 223.52 54.61 270) (unit 1)
+    (in_bom yes) (on_board yes) (dnp no) (fields_autoplaced)
+    (property "Reference" "#FLG02" (at 225.425 54.61 0)
+      (effects (font (size 1.27 1.27)) hide)
+    )
+    (property "Value" "PWR_FLAG" (at 227.33 54.61 90)
+      (effects (font (size 1.27 1.27)) (justify left))
+    )
+    (property "Footprint" "" (at 223.52 54.61 0)
+      (effects (font (size 1.27 1.27)) hide)
+    )
+    (property "Datasheet" "~" (at 223.52 54.61 0)
+      (effects (font (size 1.27 1.27)) hide)
+    )
+    (pin "1")
+    (instances
+      (project "leo68k"
+        (path "/33088729-b62e-4c27-bd07-0e3dd7f7f61e/3f60a7ce-0238-4481-8009-2dff3c5599e1"
+          (reference "#FLG02") (unit 1)
+        )
+      )

Commit message: updates
Connections:
- net VCC: no longer C7.1, C8.1, FB2.1, R2.1, TP6.1
- new net +5V: C7.1, C8.1, FB2.1, R2.1, TP6.1
Other:
- note added: "Powers Loader, CPU, RAM and logic FIXME: create footprint"
- note added: "Powers and USB connects UART FIXME: create footprint"
- note removed: "FIXME: create usb footprint"
- note removed: "USB connection to PC Connects and powers uart and loader"
- note removed: "USB power connection Powers CPU, RAM and logic"
- moved on the sheet: C1, C2, C3, C6, C7, C8, D1, D2, FB1, FB2, J1, J4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

Commit message: updates
Parts:
- removed R2: R, Resistor_SMD:R_0603_1608Metric, symbol Device:R
- added R15: 120, Resistor_SMD:R_0603_1608Metric, symbol Device:R
- D1: value LED -> USB_VBUS
- D2: value LED -> USB_POWER
- R1: value R -> 120; JLPCB Part C25808 -> C22787
Connections:
- net +5V: now also R15.1
- net at D2.2 (A): now also R15.2
Other:
- note added: "Green"
- note added: "Power input design from FT232RL datasheet page 19 and 20: https://datasheet.lcsc.com/szlcsc/Future-Designs-FT232RL-REEL_C8690.pdf Capacitor 10nF changed to 470nF Sugested Ferrite Bead MI0805K400R-00 40 Ohms @ 100MHz 1.5A (0805) change to 100 Ohms @ 100Mhz LED, 80% lumosity needs 15mA, 15mA is 3.15V Resistor 120 Ohm 0.1W vcc=5; i=15; vf=3.15; (vcc-vf)/(i/1000); (i/1000)*(vcc-vf) = 123 Ohms, .028 W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"
- note removed: "Power input design from FT232RL datasheet page 19 and 20: https://datasheet.lcsc.com/szlcsc/Future-Designs-FT232RL-REEL_C8690.pdf Capacitor 10nF changed to 470nF Sugested Ferrite Bead MI0805K400R-00 40 Ohms @ 100MHz 1.5A (0805) change to 100 Ohms @ 100Mhz LED is 80% lumosity needs 15mA, 15mA is 3.15V Resistor 120 Ohm 0.1W vcc=5; i=15; vf=3.15; (vcc-vf)/(i/1000); (i/1000)*(vcc-vf) = 123 Ohms, .028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"
Changed lines of the file:
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@@
+    (effects (font (size 1.27 1.27)) (justify left bottom))
+  )
+  (text "Green" (at 222.25 115.57 0)
     (effects (font (size 1.27 1.27)) (justify left bottom))
   )
@@
     (effects (font (size 1.27 1.27)) (justify left bottom))
   )
-  (text "Power input design from FT232RL datasheet page 19 and 20:\nhttps://datasheet.lcsc.com/szlcsc/Future-Designs-FT232RL-REEL_C8690.pdf\n\nCapacitor 10nF changed to 470nF\nSugested Ferrite Bead MI0805K400R-00 40 Ohms @ 100MHz 1.5A (0805) change to 100 Ohms @ 100Mhz\nLED is 80% lumosity needs 15mA, 15mA is 3.15V\nResistor 120 Ohm 0.1W\n  vcc=5; i=15; vf=3.15; (vcc-vf)/(i/1000); (i/1000)*(vcc-vf) = 123 Ohms, .028 W\n  r=120; ((vcc-vf)/r)*1000 = 15.4 mA"
+  (text "Power input design from FT232RL datasheet page 19 and 20:\nhttps://datasheet.lcsc.com/szlcsc/Future-Designs-FT232RL-REEL_C8690.pdf\n\nCapacitor 10nF changed to 470nF\nSugested Ferrite Bead MI0805K400R-00 40 Ohms @ 100MHz 1.5A (0805) change to 100 Ohms @ 100Mhz\nLED, 80% lumosity needs 15mA, 15mA is 3.15V\nResistor 120 Ohm 0.1W\n  vcc=5; i=15; vf=3.15; (vcc-vf)/(i/1000); (i/1000)*(vcc-vf) = 123 Ohms, .028 W\n  r=120; ((vcc-vf)/r)*1000 = 15.4 mA"
     (at 161.29 148.59 0)
+    (effects (font (size 1.27 1.27)) (justify left bottom))
+  )
+  (text "Green" (at 222.25 58.42 0)
     (effects (font (size 1.27 1.27)) (justify left bottom))
   )
@@
       (effects (font (size 1.27 1.27)) (justify right))
     )
-    (property "Value" "LED" (at 232.41 57.4675 90)
+    (property "Value" "USB_VBUS" (at 232.41 57.4675 90)
       (effects (font (size 1.27 1.27)) (justify right))
     )
@@
       (effects (font (size 1.27 1.27)) (justify right))
     )
-    (property "Value" "LED" (at 232.41 114.6175 90)
+    (property "Value" "USB_POWER" (at 232.41 114.6175 90)
       (effects (font (size 1.27 1.27)) (justify right))
     )
@@
         (path "/33088729-b62e-4c27-bd07-0e3dd7f7f61e/3f60a7ce-0238-4481-8009-2dff3c5599e1"
           (reference "D2") (unit 1)
-        )
-      )
-    )
-  )
-  (symbol (lib_id "Device:R") (at 228.6 104.14 0) (unit 1)
-    (in_bom yes) (on_board yes) (dnp no)
-    (property "Reference" "R2" (at 231.14 102.87 0)
-      (effects (font (size 1.27 1.27)) (justify left))
-    )
-    (property "Value" "R" (at 231.14 105.41 0)
-      (effects (font (size 1.27 1.27)) (justify left))
-    )
-    (property "Footprint" "Resistor_SMD:R_0603_1608Metric" (at 226.822 104.14 90)
-      (effects (font (size 1.27 1.27)) hide)
-    )
-    (property "Datasheet" "https://datasheet.lcsc.com/lcsc/2206010045_UNI-ROYAL-Uniroyal-Elec-0603WAF1203T5E_C25808.pdf" (at 228.6 104.14 0)
-      (effects (font (size 1.27 1.27)) hide)
-    )
-    (property "JLPCB Part" "C25808" (at 228.6 104.14 0)
-      (effects (font (size 1.27 1.27)) hide)
-    )
-    (pin "1")
-    (pin "2")
-    (instances
-      (project "leo68k"
-        (path "/33088729-b62e-4c27-bd07-0e3dd7f7f61e/3f60a7ce-0238-4481-8009-2dff3c5599e1"
-          (reference "R2") (unit 1)
         )
       )
@@
     )
   )
+  (symbol (lib_id "Device:R") (at 228.6 104.14 0) (unit 1)
+    (in_bom yes) (on_board yes) (dnp no)
+    (property "Reference" "R15" (at 231.14 102.87 0)
+      (effects (font (size 1.27 1.27)) (justify left))
+    )
+    (property "Value" "120" (at 231.14 105.41 0)
+      (effects (font (size 1.27 1.27)) (justify left))
+    )
+    (property "Footprint" "Resistor_SMD:R_0603_1608Metric" (at 226.822 104.14 90)
+      (effects (font (size 1.27 1.27)) hide)
+    )
+    (property "Datasheet" "https://datasheet.lcsc.com/lcsc/2206010130_UNI-ROYAL-Uniroyal-Elec-0603WAF1200T5E_C22787.pdf" (at 228.6 104.14 0)
+      (effects (font (size 1.27 1.27)) hide)
+    )
+    (property "JLPCB Part" "C22787" (at 228.6 104.14 0)
+      (effects (font (size 1.27 1.27)) hide)
+    )
+    (pin "1")
+    (pin "2")
+    (instances
+      (project "leo68k"
+        (path "/33088729-b62e-4c27-bd07-0e3dd7f7f61e/3f60a7ce-0238-4481-8009-2dff3c5599e1"
+          (reference "R15") (unit 1)
+        )
+      )
+    )
+  )
   (symbol (lib_id "Device:R") (at 228.6 46.99 0) (unit 1)
     (in_bom yes) (on_board yes) (dnp no)
@@
       (effects (font (size 1.27 1.27)) (justify left))
     )
-    (property "Value" "R" (at 231.14 48.26 0)
+    (property "Value" "120" (at 231.14 48.26 0)
       (effects (font (size 1.27 1.27)) (justify left))
     )
@@
       (effects (font (size 1.27 1.27)) hide)
     )
-    (property "Datasheet" "https://datasheet.lcsc.com/lcsc/2206010045_UNI-ROYAL-Uniroyal-Elec-0603WAF1203T5E_C25808.pdf" (at 228.6 46.99 0)
-      (effects (font (size 1.27 1.27)) hide)
-    )
-    (property "JLPCB Part" "C25808" (at 228.6 46.99 0)
-      (effects (font (size 1.27 1.27)) hide)
-    )
+    (property "Datasheet" "https://datasheet.lcsc.com/lcsc/2206010130_UNI-ROYAL-Uniroyal-Elec-0603WAF1200T5E_C22787.pdf" (at 228.6 46.99 0)
+      (effects (font (size 1.27 1.27)) hide)
+    )
+    (property "JLPCB Part" "C22787" (at 228.6 46.99 0)
+      (effects (font (size 1.27 1.27)) hide)
+    )
